File: Hardware/Wash_Hand_v1.2.brd (EAGLE design)
At the start: 71.1 x 48.3 mm, 27 parts, among them J1 I2C, J2 ICSP, J3 SPI, J4 INTERRUPT, J5 EXT_VCC, Q1 16.0 Mhz, U1 328P

Commit message: Hardware 1.2: Update the registers - it is 220Ohm, not 220K Ohm.
I updated the Wash_Hand_v1.2-routing but forgot the primary one.

Signed-off-by: Konrad Rzeszutek Wilk <konrad@kernel.org>
Parts:
- R1, R2, R3, R4, R5, R6, R7, R8: value 220K -> 220
Changed lines of the file:
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@@
 <attribute name="VALUE" x="38.227" y="10.16" size="1.27" layer="27" ratio="10" rot="R90"/>
 </element>
-<element name="R1" library="PCB_CLASS_PREMADE_COMPONENTS" package="RESISTOR" value="220K" x="57.15" y="11.43" smashed="yes" rot="R90">
+<element name="R1" library="PCB_CLASS_PREMADE_COMPONENTS" package="RESISTOR" value="220" x="57.15" y="11.43" smashed="yes" rot="R90">
 <attribute name="NAME" x="55.88" y="12.7" size="1.27" layer="25" rot="R90"/>
 <attribute name="VALUE" x="59.69" y="12.7" size="1.27" layer="27" rot="R90"/>
 </element>
-<element name="R2" library="PCB_CLASS_PREMADE_COMPONENTS" package="RESISTOR" value="220K" x="3.81" y="20.32" smashed="yes" rot="R90">
+<element name="R2" library="PCB_CLASS_PREMADE_COMPONENTS" package="RESISTOR" value="220" x="3.81" y="20.32" smashed="yes" rot="R90">
 <attribute name="NAME" x="2.54" y="21.59" size="1.27" layer="25" rot="R90"/>
 <attribute name="VALUE" x="6.35" y="21.59" size="1.27" layer="27" rot="R90"/>
 </element>
-<element name="R3" library="PCB_CLASS_PREMADE_COMPONENTS" package="RESISTOR" value="220K" x="16.51" y="11.43" smashed="yes" rot="R90">
+<element name="R3" library="PCB_CLASS_PREMADE_COMPONENTS" package="RESISTOR" value="220" x="16.51" y="11.43" smashed="yes" rot="R90">
 <attribute name="NAME" x="15.24" y="12.7" size="1.27" layer="25" rot="R90"/>
 <attribute name="VALUE" x="19.05" y="12.7" size="1.27" layer="27" rot="R90"/>
 </element>
-<element name="R4" library="PCB_CLASS_PREMADE_COMPONENTS" package="RESISTOR" value="220K" x="41.91" y="11.43" smashed="yes" rot="R90">
+<element name="R4" library="PCB_CLASS_PREMADE_COMPONENTS" package="RESISTOR" value="220" x="41.91" y="11.43" smashed="yes" rot="R90">
 <attribute name="NAME" x="40.64" y="12.7" size="1.27" layer="25" rot="R90"/>
 <attribute name="VALUE" x="44.45" y="12.7" size="1.27" layer="27" rot="R90"/>
 </element>
-<element name="R5" library="PCB_CLASS_PREMADE_COMPONENTS" package="RESISTOR" value="220K" x="46.99" y="11.43" smashed="yes" rot="R90">
+<element name="R5" library="PCB_CLASS_PREMADE_COMPONENTS" package="RESISTOR" value="220" x="46.99" y="11.43" smashed="yes" rot="R90">
 <attribute name="NAME" x="45.72" y="12.7" size="1.27" layer="25" rot="R90"/>
 <attribute name="VALUE" x="49.53" y="12.7" size="1.27" layer="27" rot="R90"/>
 </element>
-<element name="R6" library="PCB_CLASS_PREMADE_COMPONENTS" package="RESISTOR" value="220K" x="52.07" y="11.43" smashed="yes" rot="R90">
+<element name="R6" library="PCB_CLASS_PREMADE_COMPONENTS" package="RESISTOR" value="220" x="52.07" y="11.43" smashed="yes" rot="R90">
 <attribute name="NAME" x="50.8" y="12.7" size="1.27" layer="25" rot="R90"/>
 <attribute name="VALUE" x="54.61" y="12.7" size="1.27" layer="27" rot="R90"/>
 </element>
-<element name="R7" library="PCB_CLASS_PREMADE_COMPONENTS" package="RESISTOR" value="220K" x="11.43" y="11.43" smashed="yes" rot="R90">
+<element name="R7" library="PCB_CLASS_PREMADE_COMPONENTS" package="RESISTOR" value="220" x="11.43" y="11.43" smashed="yes" rot="R90">
 <attribute name="NAME" x="10.16" y="12.7" size="1.27" layer="25" rot="R90"/>
 <attribute name="VALUE" x="13.97" y="12.7" size="1.27" layer="27" rot="R90"/>
 </element>
-<element name="R8" library="PCB_CLASS_PREMADE_COMPONENTS" package="RESISTOR" value="220K" x="21.59" y="11.43" smashed="yes" rot="R90">
+<element name="R8" library="PCB_CLASS_PREMADE_COMPONENTS" package="RESISTOR" value="220" x="21.59" y="11.43" smashed="yes" rot="R90">
 <attribute name="NAME" x="20.32" y="12.7" size="1.27" layer="25" rot="R90"/>
 <attribute name="VALUE" x="24.13" y="12.7" size="1.27" layer="27" rot="R90"/>
