File: Hardware/Wash_Hand_v1.3.brd (EAGLE design)
At the start: 71.1 x 48.3 mm, 62 parts, among them IC1 LM358D, IC2 LP298XS, IC3 405016TSSOP, J1 I2C, J2 ICSP, J3 SPI, J5 EXT_VCC, J6 6_PIN_SERIAL_CABLEPTH, Q1 16.0 Mhz, U2 ATMEGA328P_TQFP

Commit message: Board: PIN3,5 were not connected to GND on ATMEGA328P
Ouch!

Signed-off-by: Konrad Rzeszutek Wilk <konrad@kernel.org>
Connections:
- removed net N$17: U2.5
- removed net N$19: U2.3
- net 0: now also U2.3, U2.5
Routing:
- net 0: track 335.0 -> 343.8 mm, vias 6 -> 7
Changed lines of the file:
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@@
 <wire x1="27.3558" y1="25.5778" x2="28.956" y2="27.178" width="0.2032" layer="1"/>
 <via x="28.956" y="27.178" extent="1-16" drill="0.35"/>
-<wire x1="28.956" y1="27.178" x2="34.036" y2="32.258" width="0.2032" layer="16"/>
+<wire x1="28.956" y1="27.178" x2="31.242" y2="29.464" width="0.2032" layer="16"/>
 <via x="34.036" y="32.258" extent="1-16" drill="0.35"/>
+<wire x1="31.242" y1="29.464" x2="34.036" y2="32.258" width="0.2032" layer="16"/>
 <wire x1="34.036" y1="32.258" x2="34.036" y2="35.6806" width="0.2032" layer="1"/>
 <wire x1="34.036" y1="35.6806" x2="34.144" y2="35.7886" width="0.2032" layer="1"/>
@@
 <wire x1="67.37" y1="30.353" x2="69.342" y2="32.325" width="0.2032" layer="1"/>
 <wire x1="69.342" y1="32.325" x2="69.342" y2="34.544" width="0.2032" layer="1"/>
+<contactref element="U2" pad="5"/>
+<contactref element="U2" pad="3"/>
+<wire x1="31.242" y1="29.464" x2="34.29" y2="26.416" width="0.1524" layer="16"/>
+<wire x1="34.29" y1="26.416" x2="34.29" y2="25.908" width="0.1524" layer="16"/>
+<via x="34.29" y="25.908" extent="1-16" drill="0.35"/>
+<wire x1="33.344" y1="26.092" x2="33.528" y2="25.908" width="0.1524" layer="1"/>
+<wire x1="33.528" y1="25.908" x2="34.29" y2="25.908" width="0.1524" layer="1"/>
+<wire x1="34.944" y1="27.2034" x2="34.944" y2="26.054" width="0.1524" layer="1"/>
+<wire x1="34.944" y1="26.054" x2="34.798" y2="25.908" width="0.1524" layer="1"/>
+<wire x1="34.798" y1="25.908" x2="34.29" y2="25.908" width="0.1524" layer="1"/>
+<wire x1="33.344" y1="27.2034" x2="33.344" y2="26.092" width="0.1524" layer="1"/>
 </signal>
 <signal name="D0">
@@
 <wire x1="16.552" y1="35.348" x2="17.018" y2="35.814" width="0.1524" layer="1"/>
 </signal>
-<signal name="N$17">
-<contactref element="U2" pad="5"/>
-</signal>
-<signal name="N$19">
-<contactref element="U2" pad="3"/>
-</signal>
 <signal name="N$35">

Commit message: Schematic: Nothing is connected to ADC6,7 so delete the nets.
Signed-off-by: Konrad Rzeszutek Wilk <konrad@kernel.org>
Connections:
- removed net N$35: U2.22
- removed net N$36: U2.19
Changed lines of the file:
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@@
 <wire x1="16.552" y1="35.348" x2="17.018" y2="35.814" width="0.1524" layer="1"/>
-</signal>
-<signal name="N$35">
-<contactref element="U2" pad="22"/>
-</signal>
-<signal name="N$36">
-<contactref element="U2" pad="19"/>
 </signal>
 </signals>

Commit message: Schematic: Make internal D0 be on the right side of the jumper
..instead off on the left. On the board however the prior
layout was ok.

Signed-off-by: Konrad Rzeszutek Wilk <konrad@kernel.org>
Parts:
- moved JP3 0.25 mm to (61.7, 39.4)
Routing:
- net D0: track 93.8 -> 92.4 mm
Changed lines of the file:
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@@
 <attribute name="VALUE" x="27.432" y="43.688" size="0.6096" layer="27" font="vector" ratio="20" rot="R90" align="top-center"/>
 </element>
-<element name="JP3" library="SparkFun-Jumpers" library_urn="urn:adsk.eagle:library:528" package="SMT-JUMPER_2_NO_NO-SILK_ROUND" package3d_urn="urn:adsk.eagle:package:39278/1" value="ENA_INT_D0" x="61.976" y="39.37" smashed="yes">
-<attribute name="NAME" x="61.976" y="41.3385" size="0.6096" layer="25" font="vector" ratio="20" align="bottom-center"/>
-<attribute name="VALUE" x="61.976" y="37.4015" size="0.6096" layer="27" font="vector" ratio="20" align="top-center"/>
+<element name="JP3" library="SparkFun-Jumpers" library_urn="urn:adsk.eagle:library:528" package="SMT-JUMPER_2_NO_NO-SILK_ROUND" package3d_urn="urn:adsk.eagle:package:39278/1" value="ENA_INT_D0" x="61.722" y="39.37" smashed="yes">
+<attribute name="NAME" x="61.722" y="41.3385" size="0.6096" layer="25" font="vector" ratio="20" align="bottom-center"/>
+<attribute name="VALUE" x="61.722" y="37.4015" size="0.6096" layer="27" font="vector" ratio="20" align="top-center"/>
 </element>
 <element name="JP4" library="SparkFun-Jumpers" library_urn="urn:adsk.eagle:library:528" package="SMT-JUMPER_2_NO_NO-SILK_ROUND" package3d_urn="urn:adsk.eagle:package:39278/1" value="ENA_INT_SENSOR" x="68.072" y="39.37" smashed="yes">
@@
 <signal name="D0">
 <contactref element="J" pad="3"/>
-<contactref element="JP3" pad="2"/>
 <contactref element="JP3" pad="1"/>
 <contactref element="IC1" pad="1"/>
-<wire x1="63.246" y1="37.592" x2="63.246" y2="38.608" width="0.1524" layer="1"/>
-<wire x1="63.246" y1="37.592" x2="62.23" y2="36.576" width="0.1524" layer="1"/>
+<wire x1="62.23" y1="36.576" x2="63.246" y2="37.592" width="0.1524" layer="1"/>
 <wire x1="62.23" y1="36.576" x2="62.23" y2="33.274" width="0.1524" layer="1"/>
 <wire x1="65.024" y1="27.94" x2="66.421" y2="26.543" width="0.1524" layer="1"/>
@@
 <wire x1="68.58" y1="24.892" x2="58.928" y2="24.892" width="0.1524" layer="1"/>
 <wire x1="58.928" y1="24.892" x2="58.547" y2="25.273" width="0.1524" layer="1"/>
-<wire x1="63.246" y1="38.608" x2="63.246" y2="39.37" width="0.2032" layer="1"/>
-<wire x1="60.706" y1="39.37" x2="61.976" y2="39.37" width="0.2032" layer="1"/>
-<wire x1="61.976" y1="39.37" x2="63.246" y2="39.37" width="0.2032" layer="1"/>
 <wire x1="66.421" y1="26.543" x2="67.37" y2="26.543" width="0.1524" layer="1"/>
 <contactref element="U2" pad="23"/>
-<wire x1="61.976" y1="39.37" x2="59.944" y2="39.37" width="0.1524" layer="1"/>
-<wire x1="59.944" y1="39.37" x2="58.547" y2="37.973" width="0.1524" layer="1"/>
+<wire x1="58.547" y1="37.973" x2="59.944" y2="39.37" width="0.1524" layer="1"/>
 <wire x1="58.547" y1="37.973" x2="58.547" y2="29.718" width="0.1524" layer="1"/>
 <wire x1="58.547" y1="29.718" x2="58.547" y2="25.273" width="0.1524" layer="1"/>
@@
 <wire x1="57.404" y1="29.718" x2="58.547" y2="29.718" width="0.1524" layer="1"/>
 <wire x1="55.118" y1="32.004" x2="57.404" y2="29.718" width="0.1524" layer="1"/>
+<wire x1="60.452" y1="39.37" x2="59.944" y2="39.37" width="0.1524" layer="1"/>
+<contactref element="JP3" pad="2"/>
+<wire x1="63.246" y1="39.116" x2="62.992" y2="39.37" width="0.1524" layer="1"/>
+<wire x1="63.246" y1="37.592" x2="63.246" y2="39.116" width="0.1524" layer="1"/>
+<wire x1="60.452" y1="39.37" x2="62.992" y2="39.37" width="0.1524" layer="1"/>
 </signal>
 <signal name="SDA">

Commit message: Schematic: Update libraries ...
Signed-off-by: Konrad Rzeszutek Wilk <konrad@kernel.org>
Parts:
- J4: value (none) -> 9V_CONN
Changed lines of the file:
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@@
 </element>
 <element name="R11" library="darnok_common" package="1206" value="4.7K" x="21.082" y="10.922" smashed="yes" rot="R90">
-<attribute name="NAME" x="19.939" y="10.922" size="0.6096" layer="25" font="vector" ratio="20" rot="R180" align="bottom-center"/>
-<attribute name="VALUE" x="22.225" y="10.922" size="0.6096" layer="27" font="vector" ratio="20" rot="R90" align="top-center"/>
+<attribute name="NAME" x="22.225" y="10.922" size="0.6096" layer="25" font="vector" ratio="20" rot="R270" align="bottom-center"/>
+<attribute name="VALUE" x="19.177" y="10.922" size="0.6096" layer="27" font="vector" ratio="20" rot="R90" align="top-center"/>
 </element>
 <element name="JP1" library="SparkFun-Jumpers" library_urn="urn:adsk.eagle:library:528" package="SMT-JUMPER_3_2-NC_PASTE_SILK" package3d_urn="urn:adsk.eagle:package:39294/1" value="SPI_JUMPER" x="18.796" y="16.51" smashed="yes" rot="R270">
@@
 <attribute name="VALUE" x="19.939" y="44.45" size="0.6096" layer="28" font="vector" ratio="20" rot="MR90" align="top-center"/>
 </element>
-<element name="J4" library="SparkFun-Connectors" library_urn="urn:adsk.eagle:library:513" package="1X02" package3d_urn="urn:adsk.eagle:package:38039/1" value="" x="60.198" y="45.974" smashed="yes">
+<element name="J4" library="SparkFun-Connectors" library_urn="urn:adsk.eagle:library:513" package="1X02" package3d_urn="urn:adsk.eagle:package:38039/1" value="9V_CONN" x="60.198" y="45.974" smashed="yes">
 <attribute name="NAME" x="58.928" y="47.371" size="0.6096" layer="25" font="vector" ratio="20"/>
-<attribute name="VALUE" x="58.928" y="43.942" size="0.6096" layer="27" font="vector" ratio="20"/>
+<attribute name="VALUE" x="59.436" y="42.164" size="0.6096" layer="27" font="vector" ratio="20"/>
 </element>
 <element name="JP2" library="SparkFun-Jumpers" library_urn="urn:adsk.eagle:library:528" package="SMT-JUMPER_3_1-NC_PASTE_SILK" package3d_urn="urn:adsk.eagle:package:39293/1" value="9V_JUMPER" x="29.21" y="43.688" smashed="yes" rot="R270">

Commit message: Board/Schematic: Update to v1.3b_rc4
Signed-off-by: Konrad Rzeszutek Wilk <konrad@kernel.org>
Other:
- board text added: "v1.3b.rc4"
- board text removed: "v1.3b.2"
Changed lines of the file:
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@@
 <circle x="8.636" y="38.862" radius="0.254" width="0.254" layer="25"/>
 <circle x="8.636" y="38.862" radius="0.567959375" width="0.1524" layer="25"/>
-<text x="32.004" y="5.842" size="1.778" layer="26" ratio="14" rot="MR0">v1.3b.2</text>
+<text x="32.004" y="5.842" size="1.778" layer="26" ratio="14" rot="MR0">v1.3b.rc4</text>
 <text x="52.832" y="15.494" size="1.016" layer="25" ratio="14">#
 [  ]

Commit message: Board/Schematic: Change 22pf to 10pf
Which makes the crystal work..

Signed-off-by: Konrad Rzeszutek Wilk <konrad@kernel.org>
Parts:
- C1, C2: value 22pF -> 10pF
Changed lines of the file:
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@@
 </autorouter>
 <elements>
-<element name="C1" library="SparkFun-Capacitors" library_urn="urn:adsk.eagle:library:510" package="1206" package3d_urn="urn:adsk.eagle:package:37426/1" value="22pF" x="25.654" y="18.288" smashed="yes" rot="R270">
+<element name="C1" library="SparkFun-Capacitors" library_urn="urn:adsk.eagle:library:510" package="1206" package3d_urn="urn:adsk.eagle:package:37426/1" value="10pF" x="25.654" y="18.288" smashed="yes" rot="R270">
 <attribute name="NAME" x="26.67" y="18.288" size="0.6096" layer="25" font="vector" ratio="20" rot="R270" align="bottom-center"/>
 <attribute name="PROD_ID" value="CAP-10057" x="-28.956" y="-4.572" size="1.778" layer="27" rot="R270" display="off"/>
 <attribute name="VALUE" value="10uF" x="24.638" y="18.288" size="0.6096" layer="27" font="vector" ratio="20" rot="R270" align="top-center"/>
 </element>
-<element name="C2" library="SparkFun-Capacitors" library_urn="urn:adsk.eagle:library:510" package="1206" package3d_urn="urn:adsk.eagle:package:37426/1" value="22pF" x="29.718" y="18.288" smashed="yes" rot="R90">
+<element name="C2" library="SparkFun-Capacitors" library_urn="urn:adsk.eagle:library:510" package="1206" package3d_urn="urn:adsk.eagle:package:37426/1" value="10pF" x="29.718" y="18.288" smashed="yes" rot="R90">
 <attribute name="NAME" x="28.702" y="18.288" size="0.6096" layer="25" font="vector" ratio="20" rot="R90" align="bottom-center"/>
 <attribute name="PROD_ID" value="CAP-10057" x="84.328" y="46.228" size="1.778" layer="27" rot="R90" display="off"/>
